Commit message: changed rotunit fixed frame to laser_fixed
Previously, rotunit used odom_combined as a fixed frame, this was now changed.
laser_fixed was added and sits at the laser's center with the same orientation
as the base_link frame.

File: kurt_base/urdf/rotunit.urdf.xacro (robot description, xacro)
@@ -100,4 +100,24 @@
     <xacro:cylinder_inertial radius="${rotunit_turntable_radius}" length="${rotunit_turntable_length}" mass="${rotunit_turntable_mass}" />
   </link>
+ <link name="rotunit_turntable_fixed_link">
+    <visual>
+      <geometry>
+        <cylinder radius="${rotunit_turntable_radius}" length="${rotunit_turntable_length}" />
+      </geometry>
+      <material name="silver" />
+    </visual>
+    <collision>
+      <geometry>
+        <cylinder radius="${rotunit_turntable_radius}" length="${rotunit_turntable_length}" />
+      </geometry>
+    </collision>
+    <xacro:cylinder_inertial radius="${rotunit_turntable_radius}" length="${rotunit_turntable_length}" mass="${rotunit_turntable_mass}" />
+  </link>
+  <joint name="laser_fixed_joint" type="fixed">
+    <parent link="rotunit_box_link" />
+    <child link="rotunit_turntable_fixed_link" />
+    <origin xyz="0 0 ${rotunit_box_z/2 + rotunit_turntable_length/2}" rpy="${M_PI} 0 ${M_PI/2}" />
+    <axis xyz="0 0 1" />
+  </joint>
   <joint name="laser_rot_joint" type="continuous">
     <parent link="rotunit_box_link" />
@@ -149,4 +169,11 @@
     <origin xyz="${rotunit_laser_x_offset} ${-rotunit_laser_y_offset} ${-rotunit_laser_z_offset}" rpy="${M_PI/2} 0 0"/>
   </joint>
+  <joint name="rotunit_laser_fixed_joint" type="fixed">
+    <parent link="rotunit_turntable_fixed_link" />
+    <child link="laser_fixed" />
+    <origin xyz="${rotunit_laser_x_offset} ${-rotunit_laser_y_offset} ${-rotunit_laser_z_offset}" rpy="0 -${M_PI} -${M_PI/2}"/>
+  </joint>
+  <link name="laser_fixed">
+  </link>
   <gazebo>
     <controller:gazebo_ros_controller_manager name="gazebo_ros_controller_manager" plugin="libgazebo_ros_controller_manager.so">

Commit message: adapted laser topic to laser360

File: kurt_base/urdf/rotunit.urdf.xacro (robot description, xacro)
@@ -7,5 +7,5 @@
   <include filename="$(find uos_common_urdf)/common.xacro" />
   <include filename="$(find uos_common_urdf)/urdf/sick_lms200.urdf.xacro" />
-  <xacro:sick_lms200 laser_link="laser" />
+  <xacro:sick_lms200 laser_link="laser360" />
   <xacro:property name="rotunit_box_x" value="0.18" />
   <xacro:property name="rotunit_box_y" value="0.18" />
@@ -147,5 +147,5 @@
   <joint name="rotunit_laser_joint" type="fixed">
     <parent link="rotunit_turntable_link" />
-    <child link="laser" />
+    <child link="laser360" />
     <origin xyz="${rotunit_laser_x_offset} ${-rotunit_laser_y_offset} ${-rotunit_laser_z_offset}" rpy="${M_PI/2} 0 0"/>
   </joint>

Commit message: Adapted laser topic to laser360
Conflicts:
	kurt_base/urdf/rotunit.urdf.xacro

File: kurt_base/urdf/rotunit.urdf.xacro (robot description, xacro)
@@ -7,5 +7,5 @@
   <xacro:include filename="$(find uos_common_urdf)/common.xacro" />
   <xacro:include filename="$(find uos_common_urdf)/urdf/sick_lms200.urdf.xacro" />
-  <xacro:sick_lms200 laser_link="laser" />
+  <xacro:sick_lms200 laser_link="laser360" />
   <xacro:property name="rotunit_box_x" value="0.18" />
   <xacro:property name="rotunit_box_y" value="0.18" />
@@ -147,5 +147,5 @@
   <joint name="rotunit_laser_joint" type="fixed">
     <parent link="rotunit_turntable_link" />
-    <child link="laser" />
+    <child link="laser360" />
     <origin xyz="${rotunit_laser_x_offset} ${-rotunit_laser_y_offset} ${-rotunit_laser_z_offset}" rpy="${M_PI/2} 0 0"/>
   </joint>

Commit message: added missing hardware interface tag

File: kurt_base/urdf/rotunit.urdf.xacro (robot description, xacro)
@@ -158,9 +158,11 @@
   <transmission name="laser_rot_trans">
     <type>transmission_interface/SimpleTransmission</type>
-    <joint name="laser_rot_joint" />
+    <joint name="laser_rot_joint">
+       <hardwareInterface>EffortJointInterface</hardwareInterface>
+    </joint>
     <actuator name="laser_rot_motor" >
       <hardwareInterface>EffortJointInterface</hardwareInterface>
-        <mechanicalReduction>1</mechanicalReduction>
-      </actuator>
+      <mechanicalReduction>1</mechanicalReduction>
+    </actuator>
   </transmission>
 </robot>
