Commit message: kurt_base URDF: reduce friction of front + rear wheels
This improves the turning behaviour and makes it a bit more realistic.

File: kurt_base/urdf/kurt_indoor.urdf.xacro (robot description, xacro)
@@ -86,5 +86,5 @@
   <!-- inertial measurement unit for gazebo -->
   <xacro:imu_gazebo link="base_link" imu_topic="imu" update_rate="100.0" stdev="${imu_stdev}" />
-  <xacro:macro name="kurt_wheel" params="name xyz rotate_visual">
+  <xacro:macro name="kurt_wheel" params="name xyz rotate_visual friction">
     <!-- rotate_visual: 0 for right side, 1 for left side -->
     <link name="${name}_wheel_link">
@@ -120,7 +120,7 @@
         <kp  value="1000000.0" />
         <kd  value="1.0" /> -->
-      <!-- Turtlebot: -->
-      <mu1 value="10"/>
-      <mu2 value="10"/>
+      <!-- Turtlebot (friction = 10.0): -->
+      <mu1 value="${friction}"/>
+      <mu2 value="${friction}"/>
       <kp value="100000000.0"/>
       <kd value="10000.0"/>
@@ -134,10 +134,10 @@
     </joint>
   </xacro:macro>
-  <xacro:kurt_wheel name="left_front" xyz="${wheel_x_offset} ${axis_length/2} ${wheel_z_offset}" rotate_visual="1" />
-  <xacro:kurt_wheel name="left_middle" xyz="0 ${middle_axis_length/2} ${wheel_z_offset}" rotate_visual="1" />
-  <xacro:kurt_wheel name="left_rear" xyz="${-wheel_x_offset} ${axis_length/2} ${wheel_z_offset}" rotate_visual="1" />
-  <xacro:kurt_wheel name="right_front" xyz="${wheel_x_offset} ${-axis_length/2} ${wheel_z_offset}" rotate_visual="0" />
-  <xacro:kurt_wheel name="right_middle" xyz="0 ${-middle_axis_length/2} ${wheel_z_offset}" rotate_visual="0" />
-  <xacro:kurt_wheel name="right_rear" xyz="${-wheel_x_offset} ${-axis_length/2} ${wheel_z_offset}" rotate_visual="0" />
+  <xacro:kurt_wheel name="left_front" xyz="${wheel_x_offset} ${axis_length/2} ${wheel_z_offset}" rotate_visual="1" friction="1.0" />
+  <xacro:kurt_wheel name="left_middle" xyz="0 ${middle_axis_length/2} ${wheel_z_offset}" rotate_visual="1" friction="10.0" />
+  <xacro:kurt_wheel name="left_rear" xyz="${-wheel_x_offset} ${axis_length/2} ${wheel_z_offset}" rotate_visual="1" friction="1.0" />
+  <xacro:kurt_wheel name="right_front" xyz="${wheel_x_offset} ${-axis_length/2} ${wheel_z_offset}" rotate_visual="0" friction="1.0" />
+  <xacro:kurt_wheel name="right_middle" xyz="0 ${-middle_axis_length/2} ${wheel_z_offset}" rotate_visual="0" friction="10.0" />
+  <xacro:kurt_wheel name="right_rear" xyz="${-wheel_x_offset} ${-axis_length/2} ${wheel_z_offset}" rotate_visual="0" friction="1.0" />
   <!-- base_footprint is a fictitious link(frame) that is on the ground right below base_link origin,
        navigation stack dedpends on this frame -->

File: kurt_base/urdf/kurt_outdoor.urdf.xacro (robot description, xacro)
@@ -86,5 +86,5 @@
   <!-- inertial measurement unit for gazebo -->
   <xacro:imu_gazebo link="base_link" imu_topic="imu" update_rate="100.0" stdev="${imu_stdev}" />
-  <xacro:macro name="kurt_wheel" params="name xyz">
+  <xacro:macro name="kurt_wheel" params="name xyz friction">
     <link name="${name}_wheel_link">
       <visual>
@@ -110,4 +110,14 @@
       </inertial>
     </link>
+    <!-- friction parameters -->
+    <gazebo reference="${name}_wheel_link">
+      <!-- Turtlebot (friction = 10.0): -->
+      <mu1 value="${friction}"/>
+      <mu2 value="${friction}"/>
+      <kp value="100000000.0"/>
+      <kd value="10000.0"/>
+      <!-- fdir1 value="1 0 0"/ -->  <!-- see http://answers.ros.org/question/607/rotation-error-in-gazebo-simulation -->
+      <material value="Gazebo/Black" />
+    </gazebo>
     <joint name="${name}_wheel_joint" type="continuous">
       <origin xyz="${xyz}" rpy="0 0 0" />
@@ -116,14 +126,11 @@
       <axis xyz="0 1 0"/>
     </joint>
-    <gazebo reference="kurt_wheel_${name}">
-      <material value="Gazebo/Grey" />
-    </gazebo>
   </xacro:macro>
-  <xacro:kurt_wheel name="left_front" xyz="${wheel_x_offset} ${axis_length/2} ${wheel_z_offset}" />
-  <xacro:kurt_wheel name="left_middle" xyz="0 ${middle_axis_length/2} ${wheel_z_offset}" />
-  <xacro:kurt_wheel name="left_rear" xyz="${-wheel_x_offset} ${axis_length/2} ${wheel_z_offset}" />
-  <xacro:kurt_wheel name="right_front" xyz="${wheel_x_offset} ${-axis_length/2} ${wheel_z_offset}" />
-  <xacro:kurt_wheel name="right_middle" xyz="0 ${-middle_axis_length/2} ${wheel_z_offset}" />
-  <xacro:kurt_wheel name="right_rear" xyz="${-wheel_x_offset} ${-axis_length/2} ${wheel_z_offset}" />
+  <xacro:kurt_wheel name="left_front" xyz="${wheel_x_offset} ${axis_length/2} ${wheel_z_offset}" friction="1.0" />
+  <xacro:kurt_wheel name="left_middle" xyz="0 ${middle_axis_length/2} ${wheel_z_offset}" friction="10.0" />
+  <xacro:kurt_wheel name="left_rear" xyz="${-wheel_x_offset} ${axis_length/2} ${wheel_z_offset}" friction="1.0" />
+  <xacro:kurt_wheel name="right_front" xyz="${wheel_x_offset} ${-axis_length/2} ${wheel_z_offset}" friction="1.0" />
+  <xacro:kurt_wheel name="right_middle" xyz="0 ${-middle_axis_length/2} ${wheel_z_offset}" friction="10.0" />
+  <xacro:kurt_wheel name="right_rear" xyz="${-wheel_x_offset} ${-axis_length/2} ${wheel_z_offset}" friction="1.0" />
   <!-- base_footprint is a fictitious link(frame) that is on the ground right below base_link origin,
        navigation stack dedpends on this frame -->

Commit message: Add imu link to urdf

File: kurt_base/urdf/kurt_indoor.urdf.xacro (robot description, xacro)
@@ -157,3 +157,9 @@
     <child link="base_link" />
   </joint>
+  <link name="imu" />
+  <joint name="base_link_to_imu_joint" type="fixed">
+    <parent link="base_link" />
+    <child link="imu" />
+    <origin xyz="${-wheel_x_offset + .07} ${axis_length/2} 0" rpy="${M_PI} 0 ${M_PI/2}" />
+  </joint>
 </robot>
